Commit message: Update VIGIL simulation projects
- military_world/: military search-and-rescue world and the vigil_sar ROS 2 workspace (sar_ws)
- vigil/: master launcher menu that starts ONE of the three independent projects
- ros2_ws/ (agriculture) and vigil_rough_terrain_ws/ (rock terrain): current state
Build output (build/, install/, log/, generated/) is not included.

File: military_world/sar_ws/src/vigil_sar/urdf/agri_ugv.urdf.xacro (robot description, xacro)
@@ -7,5 +7,7 @@
          needs. Default 15 = the original.
        * the wheel joint torque (effort) limit is an argument: sim.launch.py passes
-         physics.drive.wheel_torque_limit (150 N.m). Default 400 = the original. -->
+         physics.drive.wheel_torque_limit (150 N.m). Default 400 = the original.
+       * collision proxies (urdf/collision_proxies.xacro) for body parts that were visual only:
+         rear body, full body width, rear tower, mast, LiDAR, thermal mast / camera (no mass change). -->
 <robot name="agri_ugv" xmlns:xacro="http://www.ros.org/wiki/xacro">
   <xacro:arg name="simulation" default="false"/>
@@ -15,4 +17,5 @@
   <xacro:arg name="controllers_file" default="$(find vigil_sar)/config/controllers.yaml"/>
   <xacro:include filename="$(find vigil_sar)/urdf/cad_geometry.xacro"/>
+  <xacro:include filename="$(find vigil_sar)/urdf/collision_proxies.xacro"/>
   <xacro:property name="standing" value="$(arg standing_angle)"/>
   <material name="aluminum"><color rgba="0.65 0.67 0.70 1"/></material>
@@ -34,4 +37,5 @@
     <xacro:cad_visual part="body"/>
     <collision><origin xyz="-0.0753 0 -0.1264"/><geometry><box size="1.0737 0.5 0.3523"/></geometry></collision>
+    <xacro:body_collision_proxies/>  <!-- vigil_sar: rear body, sides, tower, mast (collision only) -->
   </link>
   <joint name="body_reference" type="fixed"><parent link="base_footprint"/><child link="base_link"/><origin xyz="0 0 0.5872"/></joint>
@@ -99,5 +103,6 @@
   <link name="camera_optical_frame"/>
   <joint name="camera_optical_joint" type="fixed"><parent link="camera_link"/><child link="camera_optical_frame"/><origin rpy="${-pi/2} 0 ${-pi/2}"/></joint>
-  <link name="lidar_link"><xacro:inertia mass="0.8" x="0.07" y="0.07" z="0.06"/><xacro:cad_visual part="lidar" material="rubber"/></link>
+  <link name="lidar_link"><xacro:inertia mass="0.8" x="0.07" y="0.07" z="0.06"/><xacro:cad_visual part="lidar" material="rubber"/>
+    <collision name="lidar_collision"><origin xyz="-0.013 0 -0.012"/><geometry><cylinder radius="0.05" length="0.056"/></geometry></collision></link>
   <joint name="lidar_mount" type="fixed"><parent link="base_link"/><child link="lidar_link"/><origin xyz="-0.5865 0 0.497"/></joint>
   <link name="imu_link"><xacro:inertia mass="0.05" x="0.03" y="0.03" z="0.01"/></link>

File: military_world/sar_ws/src/vigil_sar/urdf/sar_sensors.xacro (robot description, xacro)
@@ -30,4 +30,5 @@
     <inertial><mass value="0.3"/><inertia ixx="0.001" ixy="0" ixz="0" iyy="0.001" iyz="0" izz="0.0002"/></inertial>
     <visual><origin xyz="0 0 ${mast_h / 2}"/><geometry><cylinder radius="0.015" length="${mast_h}"/></geometry><material name="aluminum"/></visual>
+    <collision name="thermal_mast_collision"><origin xyz="0 0 ${mast_h / 2}"/><geometry><cylinder radius="0.02" length="${mast_h}"/></geometry></collision>
   </link>
   <joint name="thermal_mast_mount" type="fixed"><parent link="base_link"/><child link="thermal_mast"/>
@@ -36,4 +37,5 @@
     <inertial><mass value="0.25"/><inertia ixx="0.0002" ixy="0" ixz="0" iyy="0.0002" iyz="0" izz="0.0002"/></inertial>
     <visual><geometry><box size="0.06 0.08 0.06"/></geometry><material name="rubber"/></visual>
+    <collision name="thermal_camera_collision"><geometry><box size="0.06 0.08 0.06"/></geometry></collision>
   </link>
   <joint name="thermal_mount" type="fixed"><parent link="base_link"/><child link="thermal_link"/>

File: ros2_ws/src/agri_ugv_description/urdf/agri_ugv.urdf.xacro (robot description, xacro)
@@ -68,4 +68,12 @@
   <link name="imu_link"><xacro:inertia mass="0.05" x="0.03" y="0.03" z="0.01"/></link>
   <joint name="imu_mount" type="fixed"><parent link="base_link"/><child link="imu_link"/><origin xyz="-0.0753 0 -0.1264"/></joint>
+  <!-- Simulated soil-moisture probe (agri_moisture_sensor.py). Visual only (no mass, no collision):
+       under the chassis between the crop row and the left tyre, so it reads soil, not plants.
+       The link origin is the probe tip, ~4 cm above the ground. -->
+  <link name="moisture_probe_link">
+    <visual><origin xyz="0 0 0.125"/><geometry><cylinder radius="0.012" length="0.25"/></geometry><material name="aluminum"/></visual>
+    <visual><origin xyz="0 0 0.01"/><geometry><sphere radius="0.02"/></geometry><material name="rubber"/></visual>
+  </link>
+  <joint name="moisture_probe_mount" type="fixed"><parent link="base_link"/><child link="moisture_probe_link"/><origin xyz="-0.10 0.30 -0.55"/></joint>
   <xacro:if value="$(arg simulation)"><xacro:include filename="$(find agri_ugv_description)/urdf/simulation.xacro"/></xacro:if>
 </robot>
